File: MacroPad.kicad_sch (KiCad schematic)
At the start: 0 parts

Commit message: Feat: Complete schematic and started pcb
Parts:
- added A1: RaspberryPi_Pico, Module:RaspberryPi_Pico_Common_Unspecified, symbol MCU_Module:RaspberryPi_Pico
- added D1, D10, D11, D12, D13, D14, D2, D3, D4, D5, D6, D7, D8, D9: D, Diode_THT:D_DO-35_SOD27_P7.62mm_Horizontal, symbol Device:D
- added D15, D16, D17, D18, D19, D20, D21, D22, D23, D24, D25, D26: SK6812MINI-E, Hackpad:SK6812MINI-E_fixed, symbol SK6812MINI-E:SK6812MINI-E
- added J1: Conn_01x04_Pin, Connector_PinHeader_1.27mm:PinHeader_1x04_P1.27mm_Vertical, symbol Connector:Conn_01x04_Pin
- added SW1, SW10, SW11, SW12, SW2, SW3, SW4, SW5, SW6, SW7, SW8, SW9: SW_Push, Button_Switch_Keyboard:SW_Cherry_MX_1.00u_PCB, symbol Switch:SW_Push
- added SW13, SW14: RotaryEncoder_Switch, Hackpad:RotaryEncoder_Alps_EC11E-Switch_Vertical_H20mm, symbol Device:RotaryEncoder_Switch
Connections:
- new net: D8.2 (A), SW8.2
- new net: D19.2 (DOUT), D20.4 (DIN)
- new net: D18.2 (DOUT), D19.4 (DIN)
- new net: D7.2 (A), SW7.2
- new net: D17.2 (DOUT), D18.4 (DIN)
- new net: D16.2 (DOUT), D17.4 (DIN)
- new net: D21.2 (DOUT), D22.4 (DIN)
- new net: D20.2 (DOUT), D21.4 (DIN)
- new net: D5.2 (A), SW5.2
- new net: D10.2 (A), SW10.2
- new net: D24.2 (DOUT), D25.4 (DIN)
- new net: D23.2 (DOUT), D24.4 (DIN)
- new net: D6.2 (A), SW6.2
- new net: D25.2 (DOUT), D26.4 (DIN)
- new net: D11.2 (A), SW11.2
- new net: D4.2 (A), SW4.2
- new net: D12.2 (A), SW12.2
- new net: D3.2 (A), SW3.2
- new net: D1.2 (A), SW1.2
- new net: D2.2 (A), SW2.2
- new net: D15.2 (DOUT), D16.4 (DIN)
- new net: D22.2 (DOUT), D23.4 (DIN)
- new net: D9.2 (A), SW9.2
- new net ARGB_DATA: A1.16 (GPIO12), D15.4 (DIN)
- new net COL0: A1.5 (GPIO3), SW1.1, SW5.1, SW9.1
- new net COL1: A1.6 (GPIO4), SW10.1, SW2.1, SW6.1
- new net COL2: A1.7 (GPIO5), SW11.1, SW3.1, SW7.1
- new net COL3: A1.9 (GPIO6), SW12.1, SW4.1, SW8.1
- new net COL4: A1.10 (GPIO7), SW13.S2, SW14.S2
- new net GND: A1.13 (GND), A1.18 (GND), A1.23 (GND), A1.28 (GND), A1.3 (GND), A1.38 (GND), A1.8 (GND), D15.3 (VSS), D16.3 (VSS), D17.3 (VSS), D18.3 (VSS), D19.3 (VSS), D20.3 (VSS), D21.3 (VSS), D22.3 (VSS), D23.3 (VSS), D24.3 (VSS), D25.3 (VSS), D26.3 (VSS), J1.4 (Pin_4), SW13.C, SW14.C
- new net OLED_SCL: A1.20 (GPIO15), J1.2 (Pin_2)
- new net OLED_SDA: A1.19 (GPIO14), J1.1 (Pin_1)
- new net REC_A1: A1.11 (GPIO8), SW13.B
- new net REC_A2: A1.12 (GPIO9), SW13.A
- new net REC_B1: A1.14 (GPIO10), SW14.B
- new net REC_B2: A1.15 (GPIO11), SW14.A
- new net REC__SW_A2: D14.2 (A), SW13.S1
- new net REC__SW_B2: D13.2 (A), SW14.S1
- new net ROW0: A1.1 (GPIO0), D1.1 (K), D13.1 (K), D2.1 (K), D3.1 (K), D4.1 (K)
- new net ROW1: A1.2 (GPIO1), D14.1 (K), D5.1 (K), D6.1 (K), D7.1 (K), D8.1 (K)
- new net ROW2: A1.4 (GPIO2), D10.1 (K), D11.1 (K), D12.1 (K), D9.1 (K)
- new net VCC: A1.40 (VBUS), D15.1 (VDD), D16.1 (VDD), D17.1 (VDD), D18.1 (VDD), D19.1 (VDD), D20.1 (VDD), D21.1 (VDD), D22.1 (VDD), D23.1 (VDD), D24.1 (VDD), D25.1 (VDD), D26.1 (VDD), J1.3 (Pin_3)
- no-connect marks 0 -> 18
Other:
- note added: "MICROCONTROLLER"
- note added: "OLED DISPLAY"
- note added: "ROTARY ENCODER"
- note added: "SWITCH ARGB"
- note added: "SWITCH MATRIX"

Commit message: Feat: Designed the PCB
Parts:
- J1: footprint Connector_PinHeader_1.27mm:PinHeader_1x04_P1.27mm_Vertical -> Connector_PinHeader_2.54mm:PinHeader_1x04_P2.54mm_Vertical
Changed lines of the file:
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@@
 			)
 		)
-		(property "Footprint" "Connector_PinHeader_1.27mm:PinHeader_1x04_P1.27mm_Vertical"
+		(property "Footprint" "Connector_PinHeader_2.54mm:PinHeader_1x04_P2.54mm_Vertical"
 			(at 101.6 175.26 0)
 			(effects

Commit message: feat: more design
Parts:
- D15, D16, D17, D18, D19, D20, D21, D22, D23, D24, D25, D26: footprint Hackpad:SK6812MINI-E_fixed -> HackPad:SK6812MINI-E_fixed
- SW13, SW14: footprint Hackpad:RotaryEncoder_Alps_EC11E-Switch_Vertical_H20mm -> HackPad:RotaryEncoder_Alps_EC11E-Switch_Vertical_H20mm
Changed lines of the file:
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@@
 			)
 		)
-		(property "Footprint" "Hackpad:SK6812MINI-E_fixed"
+		(property "Footprint" "HackPad:SK6812MINI-E_fixed"
 			(at 208.28 127 0)
 			(effects
@@
 			)
 		)
-		(property "Footprint" "Hackpad:SK6812MINI-E_fixed"
+		(property "Footprint" "HackPad:SK6812MINI-E_fixed"
 			(at 243.84 109.22 0)
 			(effects
@@
 			)
 		)
-		(property "Footprint" "Hackpad:SK6812MINI-E_fixed"
+		(property "Footprint" "HackPad:SK6812MINI-E_fixed"
 			(at 243.84 127 0)
 			(effects
@@
 			)
 		)
-		(property "Footprint" "Hackpad:SK6812MINI-E_fixed"
+		(property "Footprint" "HackPad:SK6812MINI-E_fixed"
 			(at 226.06 127 0)
 			(effects
@@
 			)
 		)
-		(property "Footprint" "Hackpad:RotaryEncoder_Alps_EC11E-Switch_Vertical_H20mm"
+		(property "Footprint" "HackPad:RotaryEncoder_Alps_EC11E-Switch_Vertical_H20mm"
 			(at 84.074 73.66 0)
 			(effects
@@
 			)
 		)
-		(property "Footprint" "Hackpad:SK6812MINI-E_fixed"
+		(property "Footprint" "HackPad:SK6812MINI-E_fixed"
 			(at 226.06 144.78 0)
 			(effects
@@
 			)
 		)
-		(property "Footprint" "Hackpad:RotaryEncoder_Alps_EC11E-Switch_Vertical_H20mm"
+		(property "Footprint" "HackPad:RotaryEncoder_Alps_EC11E-Switch_Vertical_H20mm"
 			(at 45.974 73.66 0)
 			(effects
@@
 			)
 		)
-		(property "Footprint" "Hackpad:SK6812MINI-E_fixed"
+		(property "Footprint" "HackPad:SK6812MINI-E_fixed"
 			(at 261.62 144.78 0)
 			(effects
@@
 			)
 		)
-		(property "Footprint" "Hackpad:SK6812MINI-E_fixed"
+		(property "Footprint" "HackPad:SK6812MINI-E_fixed"
 			(at 243.84 144.78 0)
 			(effects
@@
 			)
 		)
-		(property "Footprint" "Hackpad:SK6812MINI-E_fixed"
+		(property "Footprint" "HackPad:SK6812MINI-E_fixed"
 			(at 226.06 109.22 0)
 			(effects
@@
 			)
 		)
-		(property "Footprint" "Hackpad:SK6812MINI-E_fixed"
+		(property "Footprint" "HackPad:SK6812MINI-E_fixed"
 			(at 208.28 144.78 0)
 			(effects
@@
 			)
 		)
-		(property "Footprint" "Hackpad:SK6812MINI-E_fixed"
+		(property "Footprint" "HackPad:SK6812MINI-E_fixed"
 			(at 261.62 109.22 0)
 			(effects
@@
 			)
 		)
-		(property "Footprint" "Hackpad:SK6812MINI-E_fixed"
+		(property "Footprint" "HackPad:SK6812MINI-E_fixed"
 			(at 261.62 127 0)
 			(effects
@@
 			)
 		)
-		(property "Footprint" "Hackpad:SK6812MINI-E_fixed"
+		(property "Footprint" "HackPad:SK6812MINI-E_fixed"
 			(at 208.28 109.22 0)
 			(effects
